Commit message: Updated to 4-wheel ackermann model and fixed a lidar smudging issue.
NOTE: The rover is currently driving and turning very slowly. The MPPI controller's acceleration and steering sampling are too timid and need to be tuned up next.

File: model/robot.xacro (robot description, xacro)
@@ -111,24 +111,46 @@
         <xacro:inertia_wheel/>
     </link>
-    <joint name="caster_joint" type="fixed">
-        <parent link="body_link"/>
-        <child link="caster_link"/>
-        <origin xyz="${s3} 0 ${r}" rpy="0 0 0"/>
-    </joint>
-    <link name="caster_link">
-        <visual>
-            <origin rpy="0 0 0" xyz="0 0 0"/>
-            <geometry>
-                <sphere radius="${r}"/>
-            </geometry>
-        </visual>
-        <collision>
-            <origin rpy="0 0 0" xyz="0 0 0"/>
-            <geometry>
-                <sphere radius="${r}"/>
-            </geometry>
-        </collision>
-        <xacro:inertia_caster/>
-    </link>
+    <xacro:macro name="steering_knuckle" params="prefix x y">
+        <joint name="${prefix}_steer_joint" type="revolute">
+            <parent link="body_link"/>
+            <child link="${prefix}_steer_link"/>
+            <origin xyz="${x} ${y} ${r}" rpy="0 0 0"/>
+            <axis xyz="0 0 1"/>
+            <limit lower="-0.785" upper="0.785" effort="5000" velocity="5.0"/>
+            <dynamics damping="1.0" friction="2.0"/>
+        </joint>
+        <link name="${prefix}_steer_link">
+            <inertial>
+                <mass value="20.0"/>
+                <origin xyz="0 0 0" rpy="0 0 0"/>
+                <inertia ixx="0.1" ixy="0" ixz="0" iyy="0.1" iyz="0" izz="0.1"/>
+            </inertial>
+        </link>
+        <joint name="${prefix}_wheel_joint" type="continuous">
+            <parent link="${prefix}_steer_link"/>
+            <child link="${prefix}_wheel_link"/>
+            <origin xyz="0 0 0" rpy="0 0 0"/>
+            <axis xyz="0 1 0"/>
+            <limit effort="50000" velocity="10"/>
+            <dynamics damping="1.0" friction="1.0"/>
+        </joint>
+        <link name="${prefix}_wheel_link">
+            <visual>
+                <origin rpy="1.570795 0 0" xyz="0 0 0"/>
+                <geometry>
+                    <cylinder length="${d}" radius="${r}"/>
+                </geometry>
+            </visual>
+            <collision>
+                <origin rpy="1.570795 0 0" xyz="0 0 0"/>
+                <geometry>
+                    <cylinder length="${d}" radius="${r}"/>
+                </geometry>
+            </collision>
+            <xacro:inertia_wheel/>
+        </link>
+    </xacro:macro>
+    <xacro:steering_knuckle prefix="front_left" x="${s3}" y="${s4}"/>
+    <xacro:steering_knuckle prefix="front_right" x="${s3}" y="${-s4}"/>
     <joint name="lidar_joint" type="fixed">
         <origin xyz="0.0 0 ${b+r}" rpy="0 0 0"/>
@@ -166,5 +188,4 @@
         <parent link="body_link"/>
         <child link="imu_link"/>
-        <origin xyz="0 0 0" rpy="0 0 0"/>
-    </joint>
+        <origin xyz="0 0 ${s1}" rpy="0 0 0"/> </joint>
 </robot>

Commit message: Calibrate physical dimensions and estimate for safe real-world speeds

File: model/robot.xacro (robot description, xacro)
@@ -2,19 +2,15 @@
 <robot name="mobile_robot" xmlns:xacro="http://www.ros.org/wiki/xacro">
     <xacro:property name="pi_const" value="3.14159265"/>
-    <xacro:property name="a" value="1.0"  />
-    <xacro:property name="b" value="0.3" />
-    <xacro:property name="c" value="0.6"/>
-    <xacro:property name="r" value="0.15"/>
-    <xacro:property name="d" value="0.1"/>
-    <xacro:property name="s1" value="${b/2+r}"/>
-    <xacro:property name="s2" value="${2*r}"/>
-    <xacro:property name="s3" value="${2*r}"/>
-    <xacro:property name="s4" value="${c/2+d/2}"/>
-    <xacro:property name="d1" value="2710.0"/>
-    <xacro:property name="d2" value="2710.0"/>
-    <xacro:property name="d3" value="2710.0"/>
-    <xacro:property name="m1" value="${d1*a*b*c}"/>
-    <xacro:property name="m2" value="${d1*pi_const*r*r*d}"/>
-    <xacro:property name="m3" value="${d3*(4.0/3.0)*pi_const*r*r*r}"/>
+    <xacro:property name="a" value="1.1176" />
+    <xacro:property name="b" value="0.4572" />
+    <xacro:property name="c" value="0.562" />
+    <xacro:property name="r" value="0.15875" />
+    <xacro:property name="d" value="0.1016" />
+    <xacro:property name="s1" value="0.4318" />
+    <xacro:property name="s2" value="0.3429" />
+    <xacro:property name="s3" value="0.3429" />
+    <xacro:property name="s4" value="0.2794" />
+    <xacro:property name="m1" value="40.0" />
+    <xacro:property name="m2" value="3.0" />
     <xacro:property name="Ix_body" value="${(1/12)*m1*(b*b+c*c)}"/>
     <xacro:property name="Iy_body" value="${(1/12)*m1*(a*a+b*b)}"/>
@@ -22,5 +18,4 @@
     <xacro:property name="Iz_wheel" value="${0.5*m2*r*r}"/>
     <xacro:property name="I_wheel" value="${(1.0/12.0)*m2*(3.0*r*r+d*d)}"/>
-    <xacro:property name="I_caster" value="${(2.0/5.0)*m3*r*r}"/>
     <xacro:macro name="inertia_body">
         <inertial>
@@ -37,11 +32,4 @@
         </inertial>
     </xacro:macro>
-    <xacro:macro name="inertia_caster">
-        <inertial>
-        <origin rpy="0 0 0" xyz="0 0 0"/>
-        <mass value="${m3}"/>
-        <inertia ixx="${I_caster}" ixy="0.0" ixz="0.0" iyy="${I_caster}" iyz="0" izz="${I_caster}"/>
-        </inertial>
-    </xacro:macro>
     <xacro:include filename="$(find mobile_robot)/model/robot.gazebo"/>
     <link name="base_footprint"> </link>
@@ -53,5 +41,5 @@
         <visual>
             <geometry>
-                <box size="${a} ${c} ${b}"/>
+                <box size="${a} ${b} ${c}"/>
             </geometry>
         <origin rpy="0 0 0" xyz="0 0 ${s1}"/>
@@ -154,5 +142,5 @@
     <xacro:steering_knuckle prefix="front_right" x="${s3}" y="${-s4}"/>
     <joint name="lidar_joint" type="fixed">
-        <origin xyz="0.0 0 ${b+r}" rpy="0 0 0"/>
+        <origin xyz="0.0 0 ${s1 + (c/2)}" rpy="0 0 0"/>
         <parent link="body_link"/>
         <child link="lidar_link"/>

Commit message: Steering seems to be fixed and tuned the reverse behavior.

File: model/robot.xacro (robot description, xacro)
@@ -106,11 +106,11 @@
             <axis xyz="0 0 1"/>
             <limit lower="-0.785" upper="0.785" effort="5000" velocity="5.0"/>
-            <dynamics damping="1.0" friction="2.0"/>
+            <dynamics damping="0.1" friction="0.1"/>
         </joint>
         <link name="${prefix}_steer_link">
             <inertial>
-                <mass value="20.0"/>
+                <mass value="0.5"/>
                 <origin xyz="0 0 0" rpy="0 0 0"/>
-                <inertia ixx="0.1" ixy="0" ixz="0" iyy="0.1" iyz="0" izz="0.1"/>
+                <inertia ixx="0.001" ixy="0" ixz="0" iyy="0.001" iyz="0" izz="0.001"/>
             </inertial>
         </link>
